File: strobe_ds.brd (EAGLE design)
At the start: 160 x 100 mm, 38 parts, among them IC1 AT90USB162A, Q1 IRF3704S, Q2 IRF3704S, T5 BC849, T6 BC849

Commit message: Poprawki Schematów
Parts:
- C4, C5: device rcl:C0805 -> rcl:C0603
Connections:
- removed net N$11: C3.2, JP1.VBUS, R7.1
- net 5V: now also C3.2, JP1.VBUS, R7.1
- net GND: now also C1.2, C4.2, C5.2
Routing:
- net 5V: track 53.7 -> 87.0 mm, vias 0 -> 1
- net N$11: track 13.6 -> 0.00 mm
- net 12V: track 83.7 -> 79.9 mm
- net N$1: track 63.4 -> 65.4 mm
Changed lines of the file:
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@@
 <setting verticaltext="up"/>
 </settings>
-<grid distance="0.05" unitdist="inch" unit="inch" style="lines" multiple="1" display="no" altdistance="0.025" altunitdist="inch" altunit="inch"/>
+<grid distance="0.05" unitdist="inch" unit="inch" style="lines" multiple="1" display="no" altdistance="0.01" altunitdist="inch" altunit="inch"/>
 <layers>
 <layer number="1" name="Top" color="4" fill="1" visible="yes" active="yes"/>
@@
 <attribute name="OC_FARNELL" value="unknown" x="57.15" y="6.35" size="1.778" layer="27" display="off"/>
 </element>
-<element name="C4" library="rcl" package="C0805" value="22Pf" x="25.4" y="41.91"/>
-<element name="C5" library="rcl" package="C0805" value="22Pf" x="33.02" y="41.91" rot="R180"/>
+<element name="C4" library="rcl" package="C0603" value="22Pf" x="25.4" y="41.91"/>
+<element name="C5" library="rcl" package="C0603" value="22Pf" x="33.02" y="41.91" rot="R180"/>
 <element name="R8" library="rcl" package="R0805" value="10K" x="33.02" y="58.42" rot="R90"/>
 <element name="IC2" library="SparkFun-PowerIC" package="SOT223" value="" x="38.1" y="57.15"/>
@@
 <wire x1="43.18" y1="61.28" x2="43.18" y2="64.77" width="0.3048" layer="16"/>
 <wire x1="43.18" y1="64.77" x2="42.545" y2="65.405" width="0.3048" layer="16"/>
-<wire x1="42.545" y1="65.405" x2="12.065" y2="65.405" width="0.3048" layer="16"/>
-<wire x1="12.065" y1="65.405" x2="10.16" y2="63.5" width="0.3048" layer="16"/>
-<wire x1="10.16" y1="63.5" x2="10.16" y2="49.53" width="0.3048" layer="16"/>
-<wire x1="10.16" y1="49.53" x2="11.43" y2="48.26" width="0.3048" layer="16"/>
-<wire x1="11.43" y1="48.26" x2="13.97" y2="48.26" width="0.3048" layer="16"/>
+<wire x1="42.545" y1="65.405" x2="10.16" y2="65.405" width="0.3048" layer="16"/>
+<wire x1="9.525" y1="64.77" x2="9.525" y2="49.53" width="0.3048" layer="16"/>
+<wire x1="10.795" y1="48.26" x2="13.97" y2="48.26" width="0.3048" layer="16"/>
 <wire x1="16.51" y1="48.58" x2="16.19" y2="48.26" width="0.3048" layer="16"/>
 <wire x1="16.19" y1="48.26" x2="13.97" y2="48.26" width="0.3048" layer="16"/>
+<wire x1="10.16" y1="65.405" x2="9.525" y2="64.77" width="0.3048" layer="16"/>
+<wire x1="10.795" y1="48.26" x2="9.525" y2="49.53" width="0.3048" layer="16"/>
 </signal>
 <signal name="N$2">
@@
 </polygon>
 <polygon width="0.3048" layer="1" isolate="0.254">
-<vertex x="8.89" y="67.31"/>
+<vertex x="7.62" y="67.31"/>
 <vertex x="55.88" y="67.31"/>
 <vertex x="55.88" y="29.21"/>
 <vertex x="8.89" y="29.21"/>
 </polygon>
+<contactref element="C4" pad="2"/>
+<contactref element="C5" pad="2"/>
+<contactref element="C1" pad="2"/>
 </signal>
 <signal name="N$3">
@@
 <wire x1="19.45" y1="55.48" x2="17.78" y2="57.15" width="0.3048" layer="1"/>
 <wire x1="17.78" y1="57.15" x2="17.46" y2="57.15" width="0.3048" layer="1"/>
-</signal>
-<signal name="N$11">
-<contactref element="JP1" pad="VBUS"/>
-<contactref element="R7" pad="1"/>
-<contactref element="C3" pad="2"/>
-<wire x1="21.26" y1="55.92" x2="19.395" y2="57.785" width="0.3048" layer="16"/>
-<wire x1="19.395" y1="57.785" x2="15.875" y2="57.785" width="0.3048" layer="16"/>
-<wire x1="15.875" y1="57.785" x2="15.24" y2="58.42" width="0.3048" layer="16"/>
-<wire x1="15.24" y1="58.42" x2="15.24" y2="59.69" width="0.3048" layer="16"/>
-<wire x1="15.24" y1="60.01" x2="15.24" y2="59.69" width="0.3048" layer="16"/>
-<wire x1="15.24" y1="59.69" x2="16.51" y2="60.96" width="0.3048" layer="16"/>
-<wire x1="16.51" y1="60.96" x2="16.51" y2="62.865" width="0.3048" layer="16"/>
-<wire x1="16.51" y1="62.865" x2="15.875" y2="63.5" width="0.3048" layer="16"/>
-<wire x1="15.875" y1="63.5" x2="15.555" y2="63.5" width="0.3048" layer="16"/>
 </signal>
 <signal name="5V">
@@
 <wire x1="20" y1="49.53" x2="20" y2="47.62" width="0.254" layer="1"/>
 <wire x1="13.02" y1="47.625" x2="13.02" y2="50.165" width="0.3048" layer="1"/>
-<wire x1="13.02" y1="50.165" x2="13.02" y2="52.39" width="0.3048" layer="1"/>
+<wire x1="13.02" y1="50.165" x2="13.02" y2="52.07" width="0.3048" layer="1"/>
+<wire x1="13.02" y1="52.07" x2="13.02" y2="52.39" width="0.3048" layer="1"/>
 <wire x1="13.02" y1="52.39" x2="13.335" y2="52.705" width="0.3048" layer="1"/>
 <wire x1="13.335" y1="52.705" x2="18.415" y2="52.705" width="0.3048" layer="1"/>
@@
 <wire x1="20" y1="47.62" x2="19.05" y2="46.67" width="0.3048" layer="1"/>
 <wire x1="19.05" y1="46.67" x2="19.05" y2="45.4" width="0.3048" layer="1"/>
+<contactref element="JP1" pad="VBUS"/>
+<contactref element="R7" pad="1"/>
+<contactref element="C3" pad="2"/>
+<wire x1="21.26" y1="55.92" x2="19.395" y2="57.785" width="0.3048" layer="16"/>
+<wire x1="19.395" y1="57.785" x2="15.875" y2="57.785" width="0.3048" layer="16"/>
+<wire x1="15.875" y1="57.785" x2="15.24" y2="58.42" width="0.3048" layer="16"/>
+<wire x1="15.24" y1="58.42" x2="15.24" y2="59.69" width="0.3048" layer="16"/>
+<wire x1="15.24" y1="60.01" x2="15.24" y2="59.69" width="0.3048" layer="16"/>
+<wire x1="15.24" y1="59.69" x2="16.51" y2="60.96" width="0.3048" layer="16"/>
+<wire x1="16.51" y1="60.96" x2="16.51" y2="62.865" width="0.3048" layer="16"/>
+<wire x1="16.51" y1="62.865" x2="15.875" y2="63.5" width="0.3048" layer="16"/>
+<wire x1="15.875" y1="63.5" x2="15.555" y2="63.5" width="0.3048" layer="16"/>
+<via x="11.176" y="63.754" extent="1-16" drill="1.27" shape="octagon"/>
+<wire x1="15.555" y1="63.5" x2="15.24" y2="63.5" width="0.254" layer="16"/>
+<wire x1="15.24" y1="63.5" x2="15.24" y2="64.77" width="0.254" layer="16"/>
+<wire x1="15.24" y1="64.77" x2="12.192" y2="64.77" width="0.254" layer="16"/>
+<wire x1="22.4724" y1="53.975" x2="22.4724" y2="53.5874" width="0.254" layer="1"/>
+<wire x1="22.4724" y1="53.5874" x2="22.225" y2="53.34" width="0.254" layer="1"/>
+<wire x1="11.43" y1="52.705" x2="11.6205" y2="52.5145" width="0.254" layer="1"/>
+<wire x1="11.6205" y1="52.5145" x2="12.065" y2="52.07" width="0.254" layer="1"/>
+<wire x1="12.065" y1="52.07" x2="13.02" y2="52.07" width="0.254" layer="1"/>
+<wire x1="12.192" y1="64.77" x2="11.176" y2="63.754" width="0.254" layer="16"/>
+<wire x1="11.176" y1="63.754" x2="11.176" y2="52.959" width="0.254" layer="1"/>
+<wire x1="11.176" y1="52.959" x2="11.43" y2="52.705" width="0.254" layer="1"/>
 </signal>
 <signal name="N$10">
@@
 <wire x1="24.67" y1="47.72" x2="24.67" y2="51.5874" width="0.3048" layer="1"/>
 <wire x1="34.036" y1="45.72" x2="33.97" y2="45.654" width="0.3048" layer="1"/>
-<wire x1="33.97" y1="45.654" x2="33.97" y2="41.91" width="0.3048" layer="1"/>
+<wire x1="33.97" y1="45.654" x2="33.87" y2="41.91" width="0.3048" layer="1"/>
 </signal>
 <signal name="N$13">
@@
 <wire x1="23.87" y1="46.234" x2="23.87" y2="51.5874" width="0.3048" layer="1"/>
 <wire x1="24.384" y1="45.72" x2="24.45" y2="45.654" width="0.3048" layer="1"/>
-<wire x1="24.45" y1="45.654" x2="24.45" y2="41.91" width="0.3048" layer="1"/>
+<wire x1="24.45" y1="45.654" x2="24.55" y2="41.91" width="0.3048" layer="1"/>
 </signal>
 <signal name="N$14">
@@
 <wire x1="43.1038" y1="52.705" x2="41.7576" y2="52.705" width="0.8128" layer="1"/>
 <wire x1="49.53" y1="55.2958" x2="49.4792" y2="55.245" width="0.8128" layer="16"/>
-<wire x1="49.4792" y1="55.245" x2="45.72" y2="55.245" width="0.8128" layer="16"/>
 <wire x1="37.465" y1="57.32" x2="51.9" y2="57.32" width="0.3048" layer="16"/>
 <wire x1="51.9" y1="57.32" x2="52.07" y2="57.15" width="0.3048" layer="16"/>
