File: strobe_ds.sch (EAGLE design)
At the start: 38 parts, among them IC1 AT90USB162A, Q1 IRF3704S, Q2 IRF3704S, T5 BC849, T6 BC849

Commit message: Poprawki Schematów
Parts:
- C4, C5: device rcl:C-EUC0805 -> rcl:C-EUC0603
Connections:
- removed net N$11: C3.2, JP1.VBUS, R7.1
- net 5V: now also C3.2, JP1.VBUS, R7.1
- net GND: now also C1.2, C4.2, C5.2
Changed lines of the file:
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@@
 <part name="GND10" library="SparkFun-Aesthetics" deviceset="GND" device=""/>
 <part name="Q3" library="crystal" deviceset="CRYSTAL" device="SM49"/>
-<part name="C4" library="rcl" deviceset="C-EU" device="C0805" value="22Pf"/>
-<part name="C5" library="rcl" deviceset="C-EU" device="C0805" value="22Pf"/>
+<part name="C4" library="rcl" deviceset="C-EU" device="C0603" value="22Pf"/>
+<part name="C5" library="rcl" deviceset="C-EU" device="C0603" value="22Pf"/>
 <part name="GND7" library="SparkFun-Aesthetics" deviceset="GND" device=""/>
 <part name="R8" library="rcl" deviceset="R-EU_" device="R0805" value="10K"/>
@@
 </segment>
 <segment>
-<wire x1="2.54" y1="144.78" x2="0" y2="144.78" width="0.1524" layer="91"/>
+<wire x1="2.54" y1="144.78" x2="2.286" y2="144.78" width="0.1524" layer="91"/>
+<wire x1="2.286" y1="144.78" x2="0" y2="144.78" width="0.1524" layer="91"/>
 <wire x1="0" y1="144.78" x2="0" y2="137.16" width="0.1524" layer="91"/>
 <wire x1="0" y1="137.16" x2="0" y2="132.08" width="0.1524" layer="91"/>
-<wire x1="2.54" y1="137.16" x2="0" y2="137.16" width="0.1524" layer="91"/>
-<wire x1="5.08" y1="154.94" x2="0" y2="154.94" width="0.1524" layer="91"/>
+<wire x1="2.54" y1="137.16" x2="2.286" y2="137.16" width="0.1524" layer="91"/>
+<wire x1="2.286" y1="137.16" x2="0" y2="137.16" width="0.1524" layer="91"/>
+<wire x1="5.08" y1="154.94" x2="4.826" y2="154.94" width="0.1524" layer="91"/>
+<wire x1="4.826" y1="154.94" x2="0" y2="154.94" width="0.1524" layer="91"/>
 <wire x1="0" y1="154.94" x2="0" y2="144.78" width="0.1524" layer="91"/>
 <junction x="0" y="144.78"/>
 <junction x="0" y="137.16"/>
 <pinref part="GND7" gate="1" pin="GND"/>
+<pinref part="C4" gate="G$1" pin="2"/>
+<junction x="2.286" y="144.78"/>
+<pinref part="C5" gate="G$1" pin="2"/>
+<junction x="2.286" y="137.16"/>
+<pinref part="C1" gate="G$1" pin="2"/>
+<junction x="4.826" y="154.94"/>
 </segment>
 <segment>
@@
 <pinref part="IC1" gate="G$1" pin="D+"/>
 <wire x1="12.7" y1="160.02" x2="22.86" y2="160.02" width="0.1524" layer="91"/>
-</segment>
-</net>
-<net name="N$11" class="0">
-<segment>
-<pinref part="JP1" gate="G$1" pin="VBUS"/>
-<wire x1="-7.62" y1="162.56" x2="-2.54" y2="162.56" width="0.1524" layer="91"/>
-<wire x1="-2.54" y1="162.56" x2="-2.54" y2="177.8" width="0.1524" layer="91"/>
-<pinref part="R7" gate="G$1" pin="1"/>
-<pinref part="C3" gate="G$1" pin="2"/>
-<junction x="-2.54" y="177.8"/>
 </segment>
 </net>
@@
 <pinref part="C2" gate="G$1" pin="2"/>
 <junction x="20.32" y="177.8"/>
-</segment>
-<segment>
+<pinref part="JP1" gate="G$1" pin="VBUS"/>
+<wire x1="-7.62" y1="162.56" x2="-2.54" y2="162.56" width="0.1524" layer="91"/>
+<wire x1="-2.54" y1="162.56" x2="-2.54" y2="170.18" width="0.1524" layer="91"/>
+<pinref part="R7" gate="G$1" pin="1"/>
+<pinref part="C3" gate="G$1" pin="2"/>
+<junction x="-2.54" y="177.8"/>
+<wire x1="-2.54" y1="170.18" x2="-2.54" y2="177.8" width="0.1524" layer="91"/>
+<wire x1="20.32" y1="170.18" x2="-2.54" y2="170.18" width="0.1524" layer="91"/>
+<junction x="-2.54" y="170.18"/>
+<junction x="20.32" y="170.18"/>
+</segment>
+<segment>
