File: strobe_print.brd (EAGLE design)
At the start: 141 x 208 mm, 265 parts, among them IC1 AT90USB162A, IC3 AT90USB162A, IC5 AT90USB162A, IC7 AT90USB162A, Q1 IRF3704S, Q10 IRF3704S, Q11 IRF3704S, Q12 IRF3704S, Q14 IRF3704S, Q15 IRF3704S, Q16 IRF3704S, Q17 IRF3704S, Q19 IRF3704S, Q2 IRF3704S, Q20 IRF3704S, Q4 IRF3704S, Q5 IRF3704S, Q6 IRF3704S, Q7 IRF3704S, Q9 IRF3704S, T1 BC849, T10 BC849, T11 BC849, T12 BC849, T13 BC849, T14 BC849, T15 BC849, T16 BC849, T17 BC849, T18 BC849, T19 BC849, T2 BC849, T20 BC849, T21 BC849, T22 BC849, T23 BC849, T24 BC849, T25 BC849, T26 BC849, T27 BC849, T28 BC849, T29 BC849, T3 BC849, T30 BC849, T31 BC849, T32 BC849, T33 BC849, T34 BC849, T35 BC849, T36 BC849, T4 BC849, T5 BC849, T6 BC849, T7 BC849, T8 BC849, T9 BC849

Commit message: bezpiecznik out
Parts:
- removed X10, X11, X12, X13, X14, X15, X16, X17, X18, X19, X20, X9: (no value), con-ptr500:AK300/2
- added C37, C46, C55, C64: 1uF, rcl:C0805
- added C38, C39, C42, C43, C44, C45, C47, C48, C51, C52, C53, C54, C56, C57, C60, C61, C62, C63, C65, C66, C69, C70, C71, C72: 100N, rcl:C0805
- added C40, C41, C49, C50, C58, C59, C67, C68: 22Pf, rcl:C0603
- added IC10, IC13, IC16, IC19, IC22: AT90USB162A, adafruit:TQFP32-08
- added IC11, IC14, IC17, IC20, IC23: (no value), SparkFun-PowerIC:SOT223
- added IC12, IC15, IC18, IC21, IC24, IC9: LM35CZ, lm35:TO92
- added JP5, JP6, JP7, JP8: USB-B, SparkFun-Connectors:USB-B-PTH
- added LED10, LED11, LED12, LED13, LED14, LED15, LED16, LED9: (no value), led:SML0805
- added Q21, Q22, Q24, Q25, Q26, Q27, Q29, Q30, Q31, Q32, Q34, Q35, Q36, Q37, Q39, Q40: IRF3704S, transistor-power:D2PACK
- added Q23, Q28, Q33, Q38: (no value), crystal:SM49
- added R113, R114, R140, R141, R167, R168, R194, R195: 22, rcl:R0805
- added R115, R129, R142, R156, R169, R183, R196, R210: 340, rcl:R0805
- added R116, R143, R170, R197: 10K, rcl:R0805
- added R117, R118, R119, R120, R121, R122, R123, R124, R125, R126, R127, R128, R130, R131, R132, R133, R136, R137, R138, R139, R144, R145, R146, R147, R148, R149, R150, R151, R152, R153, R154, R155, R157, R158, R159, R160, R163, R164, R165, R166, R171, R172, R173, R174, R175, R176, R177, R178, R179, R180, R181, R182, R184, R185, R186, R187, R190, R191, R192, R193, R198, R199, R200, R201, R202, R203, R204, R205, R206, R207, R208, R209, R211, R212, R213, R214: (no value), rcl:R0805
- added R134, R135, R161, R162, R188, R189, R215, R216: (no value), rcl:M0805
- added T37, T38, T39, T40, T41, T42, T43, T44, T45, T46, T47, T48, T49, T50, T51, T52, T53, T54, T55, T56, T57, T58, T59, T60, T61, T62, T63, T64: BC849, transistor:SOT23
- added TP17, TP18, TP19, TP20, TP21, TP22, TP23, TP24: TPB1,27, testpad:B1,27
- added U$10, U$12, U$14, U$16, U$6, U$8: LM393, SparkFun-AnalogIC:SO08
- added U$11, U$13, U$15, U$7, U$9: MF42-10, con-amphenol:MF42-10
- IC3: value AT90USB162A -> LM35CZ; device adafruit:TQFP32-08 -> lm35:TO92
- IC4: value (none) -> AT90USB162A; device SparkFun-PowerIC:SOT223 -> adafruit:TQFP32-08
- IC5: value AT90USB162A -> (none); device adafruit:TQFP32-08 -> SparkFun-PowerIC:SOT223
- IC6: value (none) -> LM35CZ; device SparkFun-PowerIC:SOT223 -> lm35:TO92
- R102, R48, R75, R88: value (none) -> 340
- R105, R49, R63, R77, R91: value 340 -> (none)
- R107, R108, R23, R25, R53, R54, R80, R81: device rcl:R0805 -> rcl:M0805
- R32, R59, R60, R86, R87: value (none) -> 22
- R34, R61: value 22 -> 340
- R35: value 340 -> 10K
- R36, R64, R92: value 10K -> (none)
- R62, R89: value 22 -> 10K
- R90: value 22 -> (none)
- U$1, U$5: value RJ45 -> MF42-10; device RJ45:RJ45 -> con-amphenol:MF42-10
- U$2, U$4: value RJ45 -> LM393; device RJ45:RJ45 -> SparkFun-AnalogIC:SO08
- U$3: value (none) -> MF42-10; device frames:A4P-LOC -> con-amphenol:MF42-10
- X1, X2, X3, X4, X5, X6, X7, X8: value (none) -> D-SUB9-H3M09RA; device con-ptr500:AK300/2 -> con-thomas-betts:H3M09RA
- moved R111 308.8 mm to (35.3, -120.4), flipped to the bottom, turned to 270 degrees
- moved T36 308.5 mm to (21.2, -117.8), flipped to the bottom, turned to 270 degrees
- moved R110 305.7 mm to (40.5, -120.1), flipped to the bottom, turned to 270 degrees
- moved TP13 304.2 mm to (32.7, -92.7)
- moved TP14 304.2 mm to (34.0, -95.6)
- moved TP15 303.2 mm to (22.9, -92.2)
- moved T34 297.7 mm to (46.8, -118.3), flipped to the bottom, turned to 0 degrees
- moved X7 296.1 mm to (14.0, -190.7), flipped to the bottom, turned to 90 degrees
- moved TP16 288.8 mm to (106.8, -92.6)
- moved Q15 286.3 mm to (28.1, -57.5), flipped to the bottom, turned to 180 degrees
- moved Q20 286.3 mm to (102.1, -57.4), flipped to the bottom, turned to 180 degrees
- moved T35 278.8 mm to (30.3, -91.4), flipped to the bottom, turned to 0 degrees
- moved R98 271.7 mm to (113.3, -53.9), turned to 180 degrees
- moved R112 271.2 mm to (35.2, -94.3), flipped to the bottom, turned to 270 degrees
- moved T33 270.2 mm to (42.7, -91.6), flipped to the bottom, turned to 0 degrees
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Connections:
- removed net N$125 (its old number): C28.1, IC7.27
- removed net N$126 (its old number): JP4.D+, R90.1
- removed net N$127 (its old number): JP4.D-, R89.1
- removed net N$47 (its old number): JP2.D-, R33.1
- removed net N$49 (its old number): IC3.29, R34.2
- removed net N$53 (its old number): IC3.24, R36.2, TP8.TP
- removed net N$55 (its old number): R30.1, T11.2
- removed net N$57 (its old number): R38.2, T11.1
- removed net N$58 (its old number): Q9.1, R39.2, R42.2
- removed net N$59 (its old number): Q10.1, R40.2, R41.2
- removed net N$90 (its old number): LED4.A, R63.2
- removed net N$91 (its old number): C23.1, IC5.2, Q13.2
- removed net N$92 (its old number): C22.1, IC5.1, Q13.1
- removed net N$93 (its old number): IC5.24, R64.2, TP12.TP
- new net 12V4: C44.1, IC14.3, R129.1, T33.3, T34.3, T35.3, T36.3, U$9.1, U$9.2, U$9.3, U$9.4, U$9.5
- new net 12V5: C53.1, IC17.3, R156.1, T41.3, T42.3, T43.3, T44.3, U$11.1, U$11.2, U$11.3, U$11.4, U$11.5
- new net 12V6: C62.1, IC20.3, R183.1, T49.3, T50.3, T51.3, T52.3, U$13.1, U$13.2, U$13.3, U$13.4, U$13.5
- new net 12V7: C71.1, IC23.3, R210.1, T57.3, T58.3, T59.3, T60.3, U$15.1, U$15.2, U$15.3, U$15.4, U$15.5
- new net 5V4: C38.2, C39.2, C42.1, C43.1, C45.1, IC13.31, IC13.32, IC13.4, IC14.2, IC14.4, IC15.1, JP5.VBUS, R115.1, R116.1, R134.2, T37.3, T38.3, T39.3, T40.3, U$10.8, X4.9
- new net 5V5: C47.2, C48.2, C51.1, C52.1, C54.1, IC16.31, IC16.32, IC16.4, IC17.2, IC17.4, IC18.1, JP6.VBUS, R142.1, R143.1, R161.2, T45.3, T46.3, T47.3, T48.3, U$12.8, X5.9
- new net 5V6: C56.2, C57.2, C60.1, C61.1, C63.1, IC19.31, IC19.32, IC19.4, IC20.2, IC20.4, IC21.1, JP7.VBUS, R169.1, R170.1, R188.2, T53.3, T54.3, T55.3, T56.3, U$14.8, X7.9
- new net 5V7: C65.2, C66.2, C69.1, C70.1, C72.1, IC22.31, IC22.32, IC22.4, IC23.2, IC23.4, IC24.1, JP8.VBUS, R196.1, R197.1, R215.2, T61.3, T62.3, T63.3, T64.3, U$16.8, X8.9
- new net B13: IC13.6, X4.4
- new net B14: IC13.7, X4.8
- new net B15: IC13.8, X4.3
- new net B16: IC16.6, X5.4
- new net B17: IC16.7, X5.8
- new net B18: IC16.8, X5.3
- new net B19: IC19.6, X7.4
- new net B20: IC19.7, X7.8
- new net B21: IC19.8, X7.3
- new net B22: IC22.6, X8.4
- new net B23: IC22.7, X8.8
- new net B24: IC22.8, X8.3
- new net CH17: IC13.18, R117.1
- new net CH18: IC13.19, R118.1
- new net CH19: IC13.20, R123.1
- new net CH20: IC13.21, R124.1
- new net CH21: IC16.18, R144.1
- new net CH22: IC16.19, R145.1
- new net CH23: IC16.20, R150.1
- new net CH24: IC16.21, R151.1
- new net CH25: IC19.18, R171.1
- new net CH26: IC19.19, R172.1
- new net CH27: IC19.20, R177.1
- new net CH28: IC19.21, R178.1
- new net CH29: IC22.18, R198.1
- new net CH30: IC22.19, R199.1
- new net CH31: IC22.20, R204.1
- new net CH32: IC22.21, R205.1
- new net GND4: C37.2, C38.1, C39.1, C40.2, C41.2, C42.2, C43.2, C44.2, C45.2, IC13.28, IC13.3, IC14.1, IC15.3, JP5.GND, LED10.C, LED9.C, Q21.3, Q22.3, Q24.3, Q25.3, R111.1, R112.1, R121.1, R122.1, R135.1, U$10.4, U$9.11, U$9.12, U$9.8, X4.5
- new net GND5: C46.2, C47.1, C48.1, C49.2, C50.2, C51.2, C52.2, C53.2, C54.2, IC16.28, IC16.3, IC17.1, IC18.3, JP6.GND, LED11.C, LED12.C, Q26.3, Q27.3, Q29.3, Q30.3, R138.1, R139.1, R148.1, R149.1, R162.1, U$11.11, U$11.12, U$11.8, U$12.4, X5.5
- new net GND6: C55.2, C56.1, C57.1, C58.2, C59.2, C60.2, C61.2, C62.2, C63.2, IC19.28, IC19.3, IC20.1, IC21.3, JP7.GND, LED13.C, LED14.C, Q31.3, Q32.3, Q34.3, Q35.3, R165.1, R166.1, R175.1, R176.1, R189.1, U$13.11, U$13.12, U$13.8, U$14.4, X7.5
- new net GND7: C64.2, C65.1, C66.1, C67.2, C68.2, C69.2, C70.2, C71.2, C72.2, IC22.28, IC22.3, IC23.1, IC24.3, JP8.GND, LED15.C, LED16.C, Q36.3, Q37.3, Q39.3, Q40.3, R192.1, R193.1, R202.1, R203.1, R216.1, U$15.11, U$15.12, U$15.8, U$16.4, X8.5
- new net L1: Q1.2, U$1.6
- new net L10: Q12.2, U$5.9
- new net L11: Q14.2, U$5.7
- new net L12: Q15.2, U$5.10
- new net L13: Q16.2, U$7.6
- new net L14: Q17.2, U$7.9
- new net L15: Q19.2, U$7.7
- new net L16: Q20.2, U$7.10
- new net L17: Q21.2, U$9.6
- new net L18: Q22.2, U$9.9
- new net L19: Q24.2, U$9.7
- new net L2: Q2.2, U$1.9
- new net L20: Q25.2, U$9.10
- new net L21: Q26.2, U$11.6
- new net L22: Q27.2, U$11.9
- new net L23: Q29.2, U$11.7
- new net L24: Q30.2, U$11.10
- new net L25: Q31.2, U$13.6
- new net L26: Q32.2, U$13.9
- new net L27: Q34.2, U$13.7
- new net L28: Q35.2, U$13.10
- new net L29: Q36.2, U$15.6
- new net L3: Q4.2, U$1.7
- new net L30: Q37.2, U$15.9
- new net L31: Q39.2, U$15.7
- new net L32: Q40.2, U$15.10
- new net L4: Q5.2, U$1.10
- new net L5: Q6.2, U$3.6
- new net L6: Q7.2, U$3.9
- new net L7: Q9.2, U$3.7
- new net L8: Q10.2, U$3.10
- new net L9: Q11.2, U$5.6
- new net N$104: Q17.1, R83.2, R84.2
- new net N$105: C28.1, IC10.27
- new net N$106: JP4.D+, R87.1
- new net N$107: JP4.D-, R86.1
- new net N$144: LED9.A, R115.2
- new net N$145: C41.1, IC13.2, Q23.2
- new net N$146: C40.1, IC13.1, Q23.1
- new net N$161: R128.2, T40.1
- new net N$162: IC13.17, TP13.TP
- new net N$163: IC13.16, TP14.TP
- new net N$164: LED10.A, R129.2
- new net N$165: R133.2, X4.1
- new net N$166: R132.2, X4.6
- new net N$167: R131.2, X4.2
- new net N$168: R130.2, X4.7
- new net N$169: IC15.2, U$10.2
- new net N$170: R134.1, R135.2, U$10.3
- new net N$171: Q26.1, R136.2, R139.2
- new net N$172: Q27.1, R137.2, R138.2
- new net N$173: C46.1, IC16.27
- new net N$174: JP6.D+, R141.1
- new net N$175: JP6.D-, R140.1
- new net N$176: IC16.30, R140.2
- new net N$177: IC16.29, R141.2
- new net N$178: LED11.A, R142.2
- new net N$179: C50.1, IC16.2, Q28.2
- new net N$180: C49.1, IC16.1, Q28.1
- new net N$181: IC16.24, R143.2, TP18.TP
- new net N$182: R136.1, T41.2
- new net N$183: R137.1, T42.2
- new net N$184: R144.2, T41.1
- new net N$185: R145.2, T42.1
- new net N$186: Q29.1, R146.2, R149.2
- new net N$187: Q30.1, R147.2, R148.2
- new net N$188: R146.1, T43.2
- new net N$189: R147.1, T44.2
- new net N$190: R150.2, T43.1
- new net N$191: R151.2, T44.1
- new net N$192: R152.2, T45.1
- new net N$193: R153.2, T46.1
- new net N$194: R154.2, T47.1
- new net N$195: R155.2, T48.1
- new net N$196: IC16.17, TP16.TP
- new net N$197: IC16.16, TP17.TP
- new net N$198: LED12.A, R156.2
- new net N$199: R160.2, X5.1
- new net N$200: R159.2, X5.6
- new net N$201: R158.2, X5.2
- new net N$202: R157.2, X5.7
- new net N$203: IC18.2, U$12.2
- new net N$204: R161.1, R162.2, U$12.3
- new net N$205: Q31.1, R163.2, R166.2
- new net N$206: Q32.1, R164.2, R165.2
- new net N$207: C55.1, IC19.27
- new net N$208: JP7.D+, R168.1
- new net N$209: JP7.D-, R167.1
- new net N$210: IC19.30, R167.2
- new net N$211: IC19.29, R168.2
- new net N$212: LED13.A, R169.2
- new net N$213: C59.1, IC19.2, Q33.2
- new net N$214: C58.1, IC19.1, Q33.1
- new net N$215: IC19.24, R170.2, TP21.TP
- new net N$216: R163.1, T49.2
- new net N$217: R164.1, T50.2
- new net N$218: R171.2, T49.1
- new net N$219: R172.2, T50.1
- new net N$220: Q34.1, R173.2, R176.2
- new net N$221: Q35.1, R174.2, R175.2
- new net N$222: R173.1, T51.2
- new net N$223: R174.1, T52.2
- new net N$224: R177.2, T51.1
- new net N$225: R178.2, T52.1
- new net N$226: R179.2, T53.1
- new net N$227: R180.2, T54.1
- new net N$228: R181.2, T55.1
- new net N$229: R182.2, T56.1
- new net N$230: IC19.17, TP19.TP
- new net N$231: IC19.16, TP20.TP
- new net N$232: LED14.A, R183.2
- new net N$233: R187.2, X7.1
- new net N$234: R186.2, X7.6
- new net N$235: R185.2, X7.2
- new net N$236: R184.2, X7.7
- new net N$237: IC21.2, U$14.2
- new net N$238: R188.1, R189.2, U$14.3
- new net N$239: Q36.1, R190.2, R193.2
- new net N$240: Q37.1, R191.2, R192.2
- new net N$241: C64.1, IC22.27
- new net N$242: JP8.D+, R195.1
- new net N$243: JP8.D-, R194.1
- new net N$244: IC22.30, R194.2
- new net N$245: IC22.29, R195.2
- new net N$246: LED15.A, R196.2
- new net N$247: C68.1, IC22.2, Q38.2
- new net N$248: C67.1, IC22.1, Q38.1
- new net N$249: IC22.24, R197.2, TP24.TP
- new net N$250: R190.1, T57.2
- new net N$251: R191.1, T58.2
- new net N$252: R198.2, T57.1
- new net N$253: R199.2, T58.1
- new net N$254: Q39.1, R200.2, R203.2
- new net N$255: Q40.1, R201.2, R202.2
- new net N$256: R200.1, T59.2
- new net N$257: R201.1, T60.2
- new net N$258: R204.2, T59.1
- new net N$259: R205.2, T60.1
- new net N$260: R206.2, T61.1
- new net N$261: R207.2, T62.1
- new net N$262: R208.2, T63.1
- new net N$263: R209.2, T64.1
- new net N$264: IC22.17, TP22.TP
- new net N$265: IC22.16, TP23.TP
- new net N$266: LED16.A, R210.2
- new net N$267: R214.2, X8.1
- new net N$268: R213.2, X8.6
- new net N$269: R212.2, X8.2
- new net N$270: R211.2, X8.7
- new net N$271: IC24.2, U$16.2
- new net N$272: R215.1, R216.2, U$16.3
- new net N$54: R42.2, T11.1
- new net N$62: LED3.A, R48.2
- new net N$64: R51.2, X1.6
- new net N$65: R50.2, X1.2
- new net N$66: R49.2, X1.7
- new net N$67: IC6.2, U$4.2
- new net N$68: R53.1, R54.2, U$4.3
- new net O21: R157.1, T48.2
- new net O22: R158.1, T47.2
- new net O23: R159.1, T46.2
- new net O24: R160.1, T45.2
- new net O25: R184.1, T56.2
- new net O26: R185.1, T55.2
- new net O27: R186.1, T54.2
- new net O28: R187.1, T53.2
- new net O29: R211.1, T64.2
- new net O30: R212.1, T63.2
- new net O31: R213.1, T62.2
- new net O32: R214.1, T61.2
- new net T21: IC13.12, R125.1
- new net T22: IC13.11, R126.1
- new net T23: IC13.10, R127.1
- new net T24: IC13.9, R128.1
- new net T25: IC13.5
- new net T26: IC16.12, R152.1
- new net T27: IC16.11, R153.1
- new net T28: IC16.10, R154.1
- new net T29: IC16.9, R155.1
- new net T30: IC16.5
- new net T31: IC19.12, R179.1
- new net T32: IC19.11, R180.1
- new net T33: IC19.10, R181.1
- new net T34: IC19.9, R182.1
- new net T35: IC19.5
- new net T36: IC22.12, R206.1
- new net T37: IC22.11, R207.1
- new net T38: IC22.10, R208.1
- new net T39: IC22.9, R209.1
- new net T40: IC22.5
- new net TEMP: IC1.15, U$2.1
- new net TEMP1: IC4.15, U$4.1
- new net TEMP2: IC7.15, U$6.1
- new net TEMP3: IC10.15, U$8.1
- new net TEMP4: IC13.15, U$10.1
- new net TEMP5: IC16.15, U$12.1
- new net TEMP6: IC19.15, U$14.1
- new net TEMP7: IC22.15, U$16.1
- net 12V: now also U$1.1, U$1.2, U$1.3, U$1.4, U$1.5; no longer X1.2, X2.2, X3.2, X4.2, X5.2
- net 12V1: now also IC5.3, R48.1, T9.3, U$3.1, U$3.2, U$3.3, U$3.4, U$3.5; no longer IC4.3, R49.1, T13.3, X10.2, X6.2, X7.2, X8.2, X9.2
- net 12V2: now also IC8.3, R75.1, T17.3, T18.3, U$5.1, U$5.2, U$5.3, U$5.4, U$5.5; no longer IC6.3, R77.1, T21.3, T22.3, X11.2, X12.2, X13.2, X14.2, X15.2
- net 12V3: now also IC11.3, R102.1, T25.3, T26.3, T27.3, U$7.1, U$7.2, U$7.3, U$7.4, U$7.5; no longer IC8.3, R105.1, T29.3, T30.3, T31.3, X16.2, X17.2, X18.2, X19.2, X20.2
- net 5V: now also IC3.1, R23.2, U$2.8, X6.9; no longer R27.2, T9.3, U$1.8
- net 5V1: now also IC4.31, IC4.32, IC5.2, IC5.4, IC6.1, R34.1, R53.2, T13.3, U$4.8, X1.9; no longer IC3.31, IC3.32, IC3.4, IC4.2, R36.1, R56.2, T17.3, T18.3, U$2.8
- net 5V2: now also IC7.31, IC7.32, IC7.4, IC8.2, IC8.4, IC9.1, R61.1, R62.1, R80.2, T21.3, T22.3, U$6.8, X2.9; no longer IC5.31, IC5.32, IC5.4, IC6.2, IC6.4, R63.1, R64.1, R84.2, T25.3, T26.3, T27.3, U$4.8
- net 5V3: now also IC10.31, IC10.32, IC10.4, IC11.2, IC11.4, IC12.1, R107.2, R88.1, R89.1, T29.3, T30.3, T31.3, U$8.8, X3.9; no longer IC7.31, IC7.32, IC7.4, IC8.2, IC8.4, R112.2, R91.1, R92.1, T33.3, T34.3, T35.3, T36.3, U$5.8
- net B1: now also X6.4; no longer U$1.7
- net B10: now also IC10.6, X3.4; no longer IC7.6, U$5.7
- net B11: now also IC10.7, X3.8; no longer IC7.7, U$5.6
- net B12: now also IC10.8, X3.3; no longer IC7.8, U$5.5
- net B2: now also X6.8; no longer U$1.6
- net B3: now also X6.3; no longer U$1.5
- net B4: now also IC4.6, X1.4; no longer IC3.6, U$2.7
- net B5: now also IC4.7, X1.8; no longer IC3.7, U$2.6
- net B6: now also IC4.8, X1.3; no longer IC3.8, U$2.5
- net B7: now also IC7.6, X2.4; no longer IC5.6, U$4.7
- net B8: now also IC7.7, X2.8; no longer IC5.7, U$4.6
- net B9: now also IC7.8, X2.3; no longer IC5.8, U$4.5
- net CH10: now also IC7.19, R64.1; no longer IC5.19, R66.1
- net CH11: now also IC7.20, R69.1; no longer IC5.20, R71.1
- net CH12: now also IC7.21, R70.1; no longer IC5.21, R72.1
- net CH13: now also IC10.18, R90.1; no longer IC7.18, R93.1
- net CH14: now also IC10.19, R91.1; no longer IC7.19, R94.1
- net CH15: now also IC10.20, R96.1; no longer IC7.20, R99.1
- net CH16: now also IC10.21, R97.1; no longer IC7.21, R100.1
- net CH5: now also IC4.18, R36.1; no longer IC3.18, R37.1
- net CH6: now also IC4.19, R37.1; no longer IC3.19, R38.1
- net CH7: now also IC4.20, R42.1; no longer IC3.20, R43.1
- net CH8: now also IC4.21, R43.1; no longer IC3.21, R44.1
- net CH9: now also IC7.18, R63.1; no longer IC5.18, R65.1
- net GND: now also IC3.3, R25.1, U$1.11, U$1.12, U$1.8, U$2.4, X6.5; no longer U$1.L1-, U$1.L2-, U$1.SH1, U$1.SH2, X3.1
- net GND1: now also IC4.28, IC4.3, IC5.1, IC6.3, R30.1, R40.1, R54.1, U$3.11, U$3.12, U$3.8, U$4.4, X1.5; no longer IC3.28, IC3.3, IC4.1, R32.1, R42.1, U$2.L1-, U$2.L2-, U$2.SH1, U$2.SH2, X8.1
- net GND2: now also IC7.28, IC7.3, IC8.1, IC9.3, R57.1, R58.1, R67.1, R68.1, R81.1, U$5.11, U$5.12, U$5.8, U$6.4, X2.5; no longer IC5.28, IC5.3, IC6.1, R59.1, R60.1, R69.1, R70.1, U$4.L1-, U$4.L2-, U$4.SH1, U$4.SH2, X13.1
- net GND3: now also IC10.28, IC10.3, IC11.1, IC12.3, R108.1, R84.1, R85.1, R94.1, R95.1, U$7.11, U$7.12, U$7.8, U$8.4, X3.5; no longer IC7.28, IC7.3, IC8.1, R87.1, R88.1, R97.1, R98.1, U$5.L1-, U$5.L2-, U$5.SH1, U$5.SH2, X18.1
- net N$100: now also R76.2, X2.7; no longer Q14.2, X14.1
- net N$101: now also IC9.2, U$6.2; no longer Q15.2, X15.1
- net N$102: now also R80.1, R81.2, U$6.3; no longer R67.1, T21.2
- net N$103: now also Q16.1, R82.2, R85.2; no longer R68.1, T22.2
- net N$108: now also IC10.30, R86.2; no longer R75.2, T25.1
- net N$109: now also IC10.29, R87.2; no longer R76.2, T26.1
- net N$110: now also LED7.A, R88.2; no longer IC5.17, TP9.TP
- net N$111: now also C32.1, IC10.2, Q18.2; no longer IC5.16, TP10.TP
- net N$112: now also C31.1, IC10.1, Q18.1; no longer IC5.15, TP11.TP
- net N$113: now also IC10.24, R89.2, TP12.TP; no longer LED5.A, R77.2
- net N$114: now also R82.1, T25.2; no longer R82.2, T27.1
- net N$115: now also R83.1, T26.2; no longer R81.2, U$4.1
- net N$116: now also R90.2, T25.1; no longer R80.2, U$4.2
- net N$117: now also R91.2, T26.1; no longer R79.2, U$4.3
- net N$118: now also Q19.1, R92.2, R95.2; no longer R78.2, U$4.4
- net N$119: now also Q20.1, R93.2, R94.2; no longer R84.1, U$4.L1+
- net N$120: now also R92.1, T27.2; no longer R83.1, U$4.L2+
- net N$121: now also R93.1, T28.2; no longer Q16.1, R85.2, R88.2
- net N$122: now also R96.2, T27.1; no longer Q17.1, R86.2, R87.2
- net N$123: now also R97.2, T28.1; no longer Q16.2, X16.1
- net N$124: now also R98.2, T29.1; no longer Q17.2, X17.1
- net N$128: now also IC10.17, TP10.TP; no longer IC7.30, R89.2
- net N$129: now also IC10.16, TP11.TP; no longer IC7.29, R90.2
- net N$130: now also LED8.A, R102.2; no longer LED7.A, R91.2
- net N$131: now also R106.2, X3.1; no longer C32.1, IC7.2, Q18.2
- net N$132: now also R105.2, X3.6; no longer C31.1, IC7.1, Q18.1
- net N$133: now also R104.2, X3.2; no longer IC7.24, R92.2, TP16.TP
- net N$134: now also R103.2, X3.7; no longer R85.1, T28.2
- net N$135: now also IC12.2, U$8.2; no longer R86.1, T29.2
- net N$136: now also R107.1, R108.2, U$8.3; no longer R93.2, T28.1
- net N$137: now also Q21.1, R109.2, R112.2; no longer R94.2, T29.1
- net N$138: now also Q22.1, R110.2, R111.2; no longer Q19.1, R95.2, R98.2
- net N$139: now also C37.1, IC13.27; no longer Q20.1, R96.2, R97.2
- net N$140: now also JP5.D+, R114.1; no longer Q19.2, X19.1
- net N$141: now also JP5.D-, R113.1; no longer Q20.2, X20.1
- net N$142: now also IC13.30, R113.2; no longer R95.1, T30.2
- net N$143: now also IC13.29, R114.2; no longer R96.1, T31.2
- net N$147: now also IC13.24, R116.2, TP15.TP; no longer R102.2, T33.1
- net N$148: now also R109.1, T33.2; no longer R103.2, T34.1
- net N$149: now also R110.1, T34.2; no longer R104.2, T35.1
- net N$150: now also R117.2, T33.1; no longer IC7.17, TP13.TP
- net N$151: now also R118.2, T34.1; no longer IC7.16, TP14.TP
- net N$152: now also Q24.1, R119.2, R122.2; no longer IC7.15, TP15.TP
- net N$153: now also Q25.1, R120.2, R121.2; no longer LED8.A, R105.2
- net N$154: now also R119.1, T35.2; no longer R110.2, T36.1
- net N$155: now also R120.1, T36.2; no longer R109.2, U$5.1
- net N$156: now also R123.2, T35.1; no longer R108.2, U$5.2
- net N$157: now also R124.2, T36.1; no longer R107.2, U$5.3
- net N$158: now also R125.2, T37.1; no longer R106.2, U$5.4
- net N$159: now also R126.2, T38.1; no longer R112.1, U$5.L1+
- net N$16: now also Q6.1, R27.2, R31.2; no longer Q4.2, X4.1
- net N$160: now also R127.2, T39.1; no longer R111.1, U$5.L2+
- net N$17: now also Q7.1, R29.2, R30.2; no longer Q5.2, X5.1
- net N$26: now also R20.2, X6.1; no longer R27.1, U$1.L1+
- net N$3: now also IC3.2, U$2.2; no longer Q1.2, X1.1
- net N$32: now also C10.1, IC4.27; no longer IC1.15, TP3.TP
- net N$33: now also R17.2, X6.6; no longer R25.1, U$1.L2+
- net N$35: now also R16.2, X6.2; no longer Q6.1, R29.2, R32.2
- net N$36: now also R15.2, X6.7; no longer Q7.1, R30.2, R31.2
- net N$38: now also JP2.D+, R33.1; no longer Q6.2, X6.1
- net N$39: now also JP2.D-, R32.1; no longer R23.2, T9.1
- net N$4: now also R23.1, R25.2, U$2.3; no longer Q2.2, X2.1
- net N$40: now also IC4.30, R32.2; no longer Q7.2, X7.1
- net N$41: now also IC4.29, R33.2; no longer R20.2, U$1.1
- net N$42: now also LED2.A, R34.2; no longer R17.2, U$1.2
- net N$43: now also C14.1, IC4.2, Q8.2; no longer R16.2, U$1.3
- net N$44: now also C13.1, IC4.1, Q8.1; no longer R15.2, U$1.4
- net N$45: now also IC4.24, R35.2, TP6.TP; no longer C10.1, IC3.27
- net N$46: now also R27.1, T9.2; no longer JP2.D+, R34.1
- net N$48: now also R36.2, T9.1; no longer IC3.30, R33.2
- net N$50: now also Q9.1, R38.2, R41.2; no longer LED2.A, R35.2
- net N$51: now also Q10.1, R39.2, R40.2; no longer C14.1, IC3.2, Q8.2
- net N$52: now also R38.1, T11.2; no longer C13.1, IC3.1, Q8.1
- net N$60: now also IC4.17, TP3.TP; no longer Q9.2, X9.1
- net N$61: now also IC4.16, TP5.TP; no longer Q10.2, X10.1
- net N$63: now also R52.2, X1.1; no longer R40.1, T13.2
- net N$69: now also Q11.1, R55.2, R58.2; no longer R48.2, T17.1
- net N$70: now also Q12.1, R56.2, R57.2; no longer IC3.17, TP5.TP
- net N$71: now also C19.1, IC7.27; no longer IC3.16, TP6.TP
- net N$72: now also JP3.D+, R60.1; no longer IC3.15, TP7.TP
- net N$73: now also JP3.D-, R59.1; no longer LED3.A, R49.2
- net N$74: now also IC7.30, R59.2; no longer R54.2, T18.1
- net N$75: now also IC7.29, R60.2; no longer R53.2, U$2.1
- net N$76: now also LED4.A, R61.2; no longer R52.2, U$2.2
- net N$77: now also C23.1, IC7.2, Q13.2; no longer R51.2, U$2.3
- net N$78: now also C22.1, IC7.1, Q13.1; no longer R50.2, U$2.4
- net N$79: now also IC7.24, R62.2, TP9.TP; no longer R56.1, U$2.L1+
- net N$80: now also T17.2; no longer U$2.L2+
- net N$81: now also R56.1, T18.2; no longer Q11.1, R57.2, R60.2
- net N$82: now also R63.2, T17.1; no longer Q12.1, R58.2, R59.2
- net N$83: now also R64.2, T18.1; no longer Q11.2, X11.1
- net N$84: now also Q14.1, R65.2, R68.2; no longer Q12.2, X12.1
- net N$85: now also Q15.1, R66.2, R67.2; no longer C19.1, IC5.27
- net N$86: now also R65.1, T19.2; no longer JP3.D+, R62.1
- net N$87: now also R66.1, T20.2; no longer JP3.D-, R61.1
- net N$88: now also R69.2, T19.1; no longer IC5.30, R61.2
- net N$89: now also R70.2, T20.1; no longer IC5.29, R62.2
- net N$94: now also IC7.17, TP7.TP; no longer R57.1, T19.2
- net N$95: now also IC7.16, TP8.TP; no longer R58.1, T20.2
- net N$96: now also LED5.A, R75.2; no longer R65.2, T19.1
- net N$97: now also R79.2, X2.1; no longer R66.2, T20.1
- net N$98: now also R78.2, X2.6; no longer Q14.1, R67.2, R70.2
- net N$99: now also R77.2, X2.2; no longer Q15.1, R68.2, R69.2
- net O10: now also R77.1, T23.2; no longer R55.2, T18.2
- net O11: now also T22.2; no longer T26.2
- net O12: now also T21.2; no longer T25.2
- net O13: now also R103.1, T32.2; no longer R80.1, T24.2
- net O14: now also R104.1, T31.2; no longer R81.1, T23.2
- net O15: now also R105.1, T30.2; no longer R83.2, T27.2
- net O16: now also T29.2; no longer T35.2
- net O17: now also R130.1, T40.2; no longer R107.1, T34.2
- net O18: now also R131.1, T39.2; no longer R108.1, T33.2
- net O19: now also R132.1, T38.2; no longer R109.1, T32.2
- net O20: now also R133.1, T37.2; no longer R111.2, T36.2
- net O5: now also R49.1, T16.2; no longer R25.2, T9.2
- net O6: now also T15.2; no longer T17.2
- net O7: now also T14.2; no longer T16.2
- net O8: now also T13.2; no longer T15.2
- net O9: now also R76.1, T24.2; no longer R53.1, T14.2
- net T10: now also IC4.5; no longer IC3.5, R54.1
- net T11: now also IC7.12, R71.1; no longer IC5.12, R73.1
- net T12: now also IC7.11, R72.1; no longer IC5.11, R74.1
- net T13: now also IC7.10, R73.1; no longer IC5.10, R75.1
- net T14: now also IC7.9, R74.1; no longer IC5.9, R76.1
- net T15: now also IC7.5; no longer IC5.5, R82.1
- net T16: now also IC10.12, R98.1; no longer IC7.12, R101.1
- net T17: now also IC10.11, R99.1; no longer IC7.11, R102.1
- net T18: now also IC10.10, R100.1; no longer IC7.10, R103.1
- net T19: now also IC10.9, R101.1; no longer IC7.9, R104.1
- net T20: now also IC10.5; no longer IC7.5, R110.1
- net T5: no longer R23.1
- net T6: now also IC4.12, R44.1; no longer IC3.12, R45.1
- net T7: now also IC4.11, R45.1; no longer IC3.11, R46.1
- net T8: now also IC4.10, R46.1; no longer IC3.10, R47.1
- net T9: now also IC4.9, R47.1; no longer IC3.9, R48.1
Routing:
- net 5V4: track 0.00 -> 270.0 mm
- net 5V7: track 0.00 -> 270.0 mm
- net 5V5: track 0.00 -> 270.0 mm
- net 5V6: track 0.00 -> 270.0 mm
- net 12V6: track 0.00 -> 193.0 mm, vias 0 -> 2
- net 12V4: track 0.00 -> 193.0 mm, vias 0 -> 2
- net 12V7: track 0.00 -> 193.0 mm, vias 0 -> 2
- net 12V5: track 0.00 -> 193.0 mm, vias 0 -> 2
- net N$40: track 89.2 -> 5.52 mm
- net N$84: track 89.2 -> 6.51 mm
- net N$124: track 89.2 -> 7.64 mm
- net N$4: track 89.2 -> 7.94 mm
- net CH22: track 0.00 -> 69.8 mm, vias 0 -> 1
- net CH30: track 0.00 -> 69.8 mm, vias 0 -> 1
- net CH18: track 0.00 -> 69.8 mm, vias 0 -> 1
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- added copper zone on layer 16, net GND
- added copper zone on layer 16, net GND1
- added copper zone on layer 16, net GND2
- added copper zone on layer 16, net GND3
- added copper zone on layer 1, net GND4
- added copper zone on layer 16, net GND4
- added copper zone on layer 1, net GND5
- added copper zone on layer 16, net GND5
- added copper zone on layer 1, net GND6
- added copper zone on layer 16, net GND6
- added copper zone on layer 1, net GND7
- added copper zone on layer 16, net GND7
Other:
- board size 141 x 208 mm -> 148.1 x 277.9 mm
- board text removed: "4-channel"
- board text removed: "LED STROBE"
