File: strobe.brd (EAGLE design)
At the start: 73.7 x 71.1 mm, 61 parts, among them IC1 AT90USB162A, IC3 LM35CZ, Q1 IRF3704S, Q2 IRF3704S, Q4 IRF3704S, Q5 IRF3704S, T1 BC849, T2 BC849, T3 BC849, T4 BC849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

Commit message: dodany reset na goldpinach, poprawka przelotki
Parts:
- removed TP4: TPB1,27, testpad:B1,27
- added JP2: M02PTH3, SparkFun-Connectors:1X02_LONGPADS
Connections:
- net GND: now also JP2.1
- net N$14: now also JP2.2; no longer TP4.TP
Routing:
- net N$14: track 5.93 -> 18.2 mm, vias 0 -> 1
- net 5V: track 270.0 -> 271.6 mm
Changed lines of the file:
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@@
 <attribute name="TP_SIGNAL_NAME" value="" x="33.799934375" y="43.4999125" size="1.778" layer="27" display="off"/>
-</element>
-<element name="TP4" library="testpad" package="B1,27" value="TPB1,27" x="22.69995625" y="46.89990625">
-<attribute name="TP_SIGNAL_NAME" value="" x="22.69995625" y="46.89990625" size="1.778" layer="27" display="off"/>
 </element>
 <element name="LED6" library="led" package="SML0805" value="" x="44.805853125" y="5.334509375"/>
@@
 <element name="R23" library="rcl" package="M0805" value="" x="61.355840625" y="44.358659375" rot="R90"/>
 <element name="R25" library="rcl" package="M0805" value="" x="61.338565625" y="39.322403125" rot="R90"/>
+<element name="JP2" library="SparkFun-Connectors" package="1X02_LONGPADS" value="M02PTH3" x="7.66891875" y="50.962059375"/>
 </elements>
 <signals>
@@
 <vertex x="5.08" y="-5.08"/>
 </polygon>
-<via x="12.7" y="48.26" extent="1-16" drill="1.3" shape="octagon"/>
-<via x="19.8882" y="2.5654" extent="1-16" drill="1.3" shape="octagon"/>
+<via x="8.147915625" y="-2.058975" extent="1-16" drill="1.3" shape="octagon"/>
+<via x="61.25145625" y="-2.1099125" extent="1-16" drill="1.3" shape="octagon"/>
 <contactref element="U$1" pad="8"/>
 <contactref element="U$1" pad="12"/>
 <contactref element="U$1" pad="11"/>
-<via x="58.116940625" y="51.034225" extent="1-16" drill="1.3" shape="octagon"/>
+<via x="60.788290625" y="51.034225" extent="1-16" drill="1.3" shape="octagon"/>
 <contactref element="U$2" pad="4"/>
 <contactref element="IC3" pad="3"/>
 <contactref element="R25" pad="1"/>
 <contactref element="IC3" pad="3"/>
+<contactref element="JP2" pad="1"/>
 </signal>
 <signal name="L1">
@@
 <wire x1="48.952759375" y1="41.222628125" x2="48.952759375" y2="49.62981875" width="0.254" layer="1"/>
 <wire x1="48.952759375" y1="49.62981875" x2="45.9016875" y2="52.680890625" width="0.254" layer="1"/>
-<wire x1="45.9016875" y1="52.680890625" x2="19.542603125" y2="52.680890625" width="0.254" layer="1"/>
-<wire x1="19.542603125" y1="52.680890625" x2="15.762734375" y2="48.901021875" width="0.254" layer="1"/>
-<wire x1="15.762734375" y1="48.901021875" x2="15.762734375" y2="45.7369625" width="0.254" layer="1"/>
 <wire x1="15.762734375" y1="45.7369625" x2="16.553696875" y2="44.946" width="0.254" layer="1"/>
 <wire x1="16.553696875" y1="44.946" x2="17.350971875" y2="44.946" width="0.254" layer="1"/>
@@
 <wire x1="51.96240625" y1="40.18761875" x2="51.96240625" y2="34.172921875" width="0.254" layer="1"/>
 <wire x1="51.96240625" y1="34.172921875" x2="53.303378125" y2="32.83195" width="0.254" layer="1"/>
+<wire x1="45.9016875" y1="52.680890625" x2="16.915784375" y2="52.680890625" width="0.3048" layer="1"/>
+<wire x1="16.915784375" y1="52.680890625" x2="15.706678125" y2="51.471784375" width="0.3048" layer="1"/>
+<wire x1="15.706678125" y1="51.471784375" x2="15.706678125" y2="45.79301875" width="0.3048" layer="1"/>
+<wire x1="15.706678125" y1="45.79301875" x2="15.762734375" y2="45.7369625" width="0.3048" layer="1"/>
 </signal>
 <signal name="N$10">
@@
 <contactref element="R8" pad="2"/>
 <wire x1="24.87" y1="45.597984375" x2="24.87" y2="45.312584375" width="0.3048" layer="1"/>
-<contactref element="TP4" pad="TP"/>
 <wire x1="24.87" y1="45.312584375" x2="23.282678125" y2="46.89990625" width="0.3048" layer="1"/>
-<wire x1="23.282678125" y1="46.89990625" x2="22.69995625" y2="46.89990625" width="0.3048" layer="1"/>
-<wire x1="22.69995625" y1="46.89990625" x2="22.649928125" y2="46.949934375" width="0.3048" layer="1"/>
-<wire x1="22.649928125" y1="46.949934375" x2="19.8998875" y2="46.949934375" width="0.3048" layer="1"/>
+<wire x1="23.282678125" y1="46.949934375" x2="19.8998875" y2="46.949934375" width="0.3048" layer="1"/>
+<contactref element="JP2" pad="2"/>
+<wire x1="23.282678125" y1="46.949934375" x2="23.282678125" y2="46.89990625" width="0.3048" layer="1"/>
+<wire x1="19.8998875" y1="46.949934375" x2="19.8998875" y2="47.310334375" width="0.3048" layer="1"/>
+<wire x1="19.8998875" y1="47.310334375" x2="19.867190625" y2="47.310334375" width="0.3048" layer="1"/>
+<wire x1="19.867190625" y1="47.310334375" x2="17.959175" y2="49.21835" width="0.3048" layer="1"/>
+<wire x1="17.959175" y1="49.21835" x2="17.959175" y2="50.416475" width="0.3048" layer="1"/>
+<wire x1="17.959175" y1="50.416475" x2="17.945559375" y2="50.430090625" width="0.3048" layer="1"/>
+<via x="17.945559375" y="50.430090625" extent="1-16" drill="0.6" shape="square"/>
+<wire x1="17.945559375" y1="50.430090625" x2="10.7408875" y2="50.430090625" width="0.3048" layer="16"/>
+<wire x1="10.7408875" y1="50.430090625" x2="10.20891875" y2="50.962059375" width="0.3048" layer="16"/>
 </signal>
 <signal name="CH3">
@@
 <contactref element="R14" pad="1"/>
 <wire x1="19.395953125" y1="27.279840625" x2="19.685" y2="27.5688875" width="0.3048" layer="16"/>
-<wire x1="19.685" y1="27.5688875" x2="19.685" y2="46.8376" width="0.3048" layer="16"/>
 <wire x1="27.27" y1="45.312584375" x2="27.2796" y2="45.322184375" width="0.254" layer="1"/>
 <wire x1="27.2796" y1="45.322184375" x2="27.2796" y2="46.9392" width="0.254" layer="1"/>
@@
 <wire x1="25.9334" y1="48.2854" x2="23.495" y2="48.2854" width="0.254" layer="1"/>
 <wire x1="23.495" y1="48.2854" x2="22.9108" y2="48.8696" width="0.254" layer="1"/>
-<wire x1="22.9108" y1="48.8696" x2="20.4978" y2="48.8696" width="0.254" layer="1"/>
-<wire x1="20.4978" y1="48.8696" x2="19.685" y2="48.0568" width="0.254" layer="1"/>
-<wire x1="19.685" y1="48.0568" x2="19.685" y2="47.371" width="0.254" layer="1"/>
-<via x="19.685" y="47.371" extent="1-16" drill="0.6" shape="octagon"/>
-<wire x1="19.685" y1="47.371" x2="19.685" y2="46.8376" width="0.254" layer="16"/>
+<wire x1="22.9108" y1="48.8696" x2="20.61591875" y2="48.8696" width="0.254" layer="1"/>
+<via x="20.532459375" y="48.81175625" extent="1-16" drill="0.6" shape="octagon"/>
+<wire x1="20.61591875" y1="48.8696" x2="20.4978" y2="48.8696" width="0.254" layer="1"/>
+<wire x1="20.532459375" y1="48.81175625" x2="20.61591875" y2="48.81175625" width="0.3048" layer="1"/>
+<wire x1="20.61591875" y1="48.81175625" x2="20.61591875" y2="48.8696" width="0.3048" layer="1"/>
+<wire x1="19.685" y1="27.5688875" x2="19.685" y2="47.964296875" width="0.3048" layer="16"/>
+<wire x1="19.685" y1="47.964296875" x2="20.532459375" y2="48.81175625" width="0.3048" layer="16"/>
 </signal>
 <signal name="12V">

Commit message: fixes + expander
Parts:
- moved U$1 17.4 mm to (59.4, 22.2), flipped to the bottom, turned to 270 degrees
- moved IC3 2.29 mm to (53.3, 33.8), flipped to the bottom
- moved JP1 0.29 mm to (10.9, 39.3)
Connections:
- net GND: now also U$1.10, U$1.6, U$1.9; no longer U$1.11, U$1.12, U$1.8
- net L1: now also U$1.12; no longer U$1.6
- net L2: now also Q4.2, U$1.11; no longer Q2.2, U$1.9
- net L3: now also Q2.2, U$1.8; no longer Q4.2, U$1.7
- net L4: now also U$1.7; no longer U$1.10
Routing:
- net L3: track 33.8 -> 16.4 mm
- net L2: track 15.2 -> 32.0 mm
- net N$16: track 0.00 -> 16.5 mm
- net N$4: track 7.94 -> 14.8 mm
- net TEMP: track 30.2 -> 32.3 mm
- net N$3: track 13.8 -> 15.5 mm
- net L1: track 16.8 -> 18.3 mm
- net 5V: track 271.6 -> 270.5 mm
- net 12V: track 193.0 -> 194.1 mm
- net L4: track 31.4 -> 32.5 mm
- net GND: vias 3 -> 5
